File: board/sniffer.kicad_pcb (KiCad board)
At the start: 2 copper layers, 302 parts, among them J1 BARREL, J10 CONN_SFP_HOST, J11 SFP_CAGE, J12 PMOD_HOST, J13 CONN_SATA_DEVICE, J14 CONN_SATA_HOST, J15 CONN_LVDS_EXPANSION_HOST, J2 32K243-40ML5, J3 BEL_FUSE_0826-1G1T-23-F, J4 XILINX_JTAG, J5 32K243-40ML5, J6 32K243-40ML5, J7 32K243-40ML5, J8 CONN_SFF8087, J9 CONN_SFF8087, Q1 SSM6N58NU, U1 OKL-T_3-W12P-C, U10 KSZ9031RN, U11 74AVCH1T45, U12 74AVCH1T45, U13 74AVCH1T45, U14 74AVCH1T45, U15 W25Q128JV, U16 FPF2498, U17 FPF2498, U18 LP2996A, U2 LTC3374-QFN, U3 MYTNA1R84RELA2RA, U4 DDR3_SODIMM, U5 XC7K70T-2FBG484, U6 ECX2-LMV-7CN-156.250-TR, U7 ECX2-LMV-3CN-125.000-TR, U8 ECX2-LMV-3CN-125.000-TR, U9 SIT1602BC-72-18S-25.000000

Commit message: Updating with progress from tonight
Parts:
- added M1: SCREW_HOLE, azonenberg_pcb:MECHANICAL_CLEARANCEHOLE_4_40, F.Cu at (43.0, 39.0)
- added M2: SCREW_HOLE, azonenberg_pcb:MECHANICAL_CLEARANCEHOLE_4_40, F.Cu at (43.0, 152.0)
- added M3: SCREW_HOLE, azonenberg_pcb:MECHANICAL_CLEARANCEHOLE_4_40, F.Cu at (185.0, 39.0)
- added M4: SCREW_HOLE, azonenberg_pcb:MECHANICAL_CLEARANCEHOLE_4_40, F.Cu at (185.0, 152.0)
- moved C1 192.7 mm to (235.0, 49.2)
- moved C10 192.7 mm to (231.2, 38.2)
- moved C12 192.7 mm to (230.0, 47.1)
- moved C13 192.7 mm to (232.5, 45.6)
- moved C14 192.7 mm to (236.6, 40.2)
- moved C143 192.7 mm to (233.7, 44.0)
- moved C144 192.7 mm to (236.6, 44.8)
- moved C15 192.7 mm to (239.1, 41.0)
- moved C16 192.7 mm to (230.4, 42.2)
- moved C18 192.7 mm to (237.5, 46.2)
- moved C19 192.7 mm to (235.0, 47.8)
- moved C2 192.7 mm to (235.6, 38.2)
- moved C20 192.7 mm to (232.5, 50.1)
- moved C21 192.7 mm to (230.4, 44.0)
- moved C22 192.7 mm to (230.4, 40.4)
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Connections:
- U5 pad AA1: /Expansion connector/LVDS13_P -> /Expansion connector/LA1_DQ5_P
- U5 pad AA3: /Expansion connector/LVDS14_P -> /Expansion connector/LA1_DQ6_P
- U5 pad AA4: /Expansion connector/LVDS15_P -> /Expansion connector/LA1_DQ7_P
- U5 pad AB1: /Expansion connector/LVDS13_N -> /Expansion connector/LA1_DQ5_N
- U5 pad AB2: /Expansion connector/LVDS14_N -> /Expansion connector/LA1_DQ6_N
- U5 pad AB3: /Expansion connector/LVDS15_N -> /Expansion connector/LA1_DQ7_N
- U5 pad K1: /Expansion connector/LA1_DQ1_P -> /Expansion connector/LVDS1_P
- U5 pad K2: /Expansion connector/LA1_DQ3_N -> /Expansion connector/LVDS3_N
- U5 pad K3: /Expansion connector/LA1_DQ3_P -> /Expansion connector/LVDS3_P
- U5 pad L1: /Expansion connector/LA1_DQ1_N -> /Expansion connector/LVDS1_N
- U5 pad L3: /Expansion connector/LA1_DQ0_P -> /Expansion connector/LVDS0_P
- U5 pad L4: /Expansion connector/LA1_DQ5_N -> /Expansion connector/LVDS5_N
- U5 pad L5: /Expansion connector/LA1_DQ5_P -> /Expansion connector/LVDS5_P
- U5 pad M1: /Expansion connector/LA1_DQ2_N -> /Expansion connector/LVDS2_N
- U5 pad M2: /Expansion connector/LA1_DQ2_P -> /Expansion connector/LVDS2_P
- U5 pad M3: /Expansion connector/LA1_DQ0_N -> /Expansion connector/LVDS0_N
- U5 pad M5: /Expansion connector/LVDS0_P -> /Expansion connector/LVDS8_P
- U5 pad N2: /Expansion connector/LA1_DQ4_N -> /Expansion connector/LVDS4_N
- U5 pad N3: /Expansion connector/LA1_DQ4_P -> /Expansion connector/LVDS4_P
- U5 pad N4: /Expansion connector/LVDS0_N -> /Expansion connector/LVDS8_N
- U5 pad N5: /Expansion connector/LVDS9_P -> /Expansion connector/LA1_DQ1_P
- U5 pad P1: /Expansion connector/LA1_DQ7_P -> /Expansion connector/LVDS7_P
- U5 pad P2: /Expansion connector/LA1_DQ6_P -> /Expansion connector/LVDS6_P
- U5 pad P4: /Expansion connector/LVDS2_P -> /Expansion connector/LVDS10_P
- U5 pad P5: /Expansion connector/LVDS9_N -> /Expansion connector/LA1_DQ1_N
- U5 pad R1: /Expansion connector/LA1_DQ7_N -> /Expansion connector/LVDS7_N
- U5 pad R2: /Expansion connector/LA1_DQ6_N -> /Expansion connector/LVDS6_N
- U5 pad R3: /Expansion connector/LVDS3_P -> /Expansion connector/LVDS11_P
- U5 pad R4: /Expansion connector/LVDS2_N -> /Expansion connector/LVDS10_N
- U5 pad T1: /Expansion connector/LVDS1_P -> /Expansion connector/LVDS9_P
- U5 pad T3: /Expansion connector/LVDS3_N -> /Expansion connector/LVDS11_N
- U5 pad T4: /Expansion connector/LVDS4_P -> /Expansion connector/LVDS12_P
- U5 pad T5: /Expansion connector/LVDS7_P -> /Expansion connector/LVDS15_P
- U5 pad U1: /Expansion connector/LVDS1_N -> /Expansion connector/LVDS9_N
- U5 pad U2: /Expansion connector/LVDS6_P -> /Expansion connector/LVDS14_P
- U5 pad U3: /Expansion connector/LVDS4_N -> /Expansion connector/LVDS12_N
- U5 pad U5: /Expansion connector/LVDS7_N -> /Expansion connector/LVDS15_N
- U5 pad V2: /Expansion connector/LVDS6_N -> /Expansion connector/LVDS14_N
- U5 pad V3: /Expansion connector/LVDS8_P -> /Expansion connector/LA1_DQ0_P
- U5 pad V4: /Expansion connector/LVDS5_P -> /Expansion connector/LVDS13_P
- U5 pad W1: /Expansion connector/LVDS11_P -> /Expansion connector/LA1_DQ3_P
- U5 pad W2: /Expansion connector/LVDS8_N -> /Expansion connector/LA1_DQ0_N
- U5 pad W4: /Expansion connector/LVDS5_N -> /Expansion connector/LVDS13_N
- U5 pad W5: /Expansion connector/LVDS10_P -> /Expansion connector/LA1_DQ2_P
- U5 pad Y1: /Expansion connector/LVDS11_N -> /Expansion connector/LA1_DQ3_N
- U5 pad Y2: /Expansion connector/LVDS12_N -> /Expansion connector/LA1_DQ4_N
- U5 pad Y3: /Expansion connector/LVDS12_P -> /Expansion connector/LA1_DQ4_P
- U5 pad Y4: /Expansion connector/LVDS10_N -> /Expansion connector/LA1_DQ2_N
Other:
- board outline added: 154 x 125 mm
- copper layers 2 -> 8
- net class Default: clearance 0.2 -> 0.1; trace_width 0.25 -> 0.16; via_dia 0.8 -> 0.45; via_drill 0.4 -> 0.25
- rule pad_to_mask_clearance: 0 -> 0.05
- rule trace_clearance: 0.2 -> 0.1
- rule trace_min: 0.2 -> 0.1
- rule via_min_drill: 0.3 -> 0.25
- rule via_min_size: 0.4 -> 0.45

Commit message: Began actual layout!
Parts:
- added G***: LOGO, w_logo:Logo_silk_polarity_center_5x1.4mm, F.Cu at (178.5, 45.0)
- C38, C39, C40, C41, R13, R16: moved to B.Cu
- moved C38 179.3 mm to (74.1, 114.1), turned to 270 degrees
- moved C40 177.8 mm to (80.0, 114.5), turned to 90 degrees
- moved C41 170.9 mm to (82.3, 120.5), turned to 270 degrees
- moved C39 140.1 mm to (84.1, 117.6)
- moved R16 135.2 mm to (105.6, 127.0), turned to 90 degrees
- moved R13 124.7 mm to (122.0, 109.5)
- moved J8 26.0 mm to (144.0, 141.0)
- moved J9 26.0 mm to (170.0, 141.0)
- moved C42 19.2 mm to (74.4, 120.8), turned to 90 degrees
- moved C43 16.1 mm to (77.0, 120.8), turned to 90 degrees
- moved C44 11.5 mm to (87.5, 121.4), turned to 180 degrees
- moved C45 10.8 mm to (87.5, 120.4), turned to 180 degrees
- moved U6 9.12 mm to (77.0, 116.8), turned to 180 degrees
- moved U7 8.20 mm to (84.0, 120.4), turned to 270 degrees
- moved U5 4.50 mm to (109.0, 116.5)
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Connections:
- U5 pad AA10: /RGMII PHY/ETH_LED2_N_1V8 -> /RGMII PHY/LA0_DQ7_P
- U5 pad AA11: /RGMII PHY/LA0_DQ3_P -> /RGMII PHY/LA0_DQ2_P
- U5 pad AA13: /RGMII PHY/LA0_DQ4_N -> /RGMII PHY/ETH_LED1_N_1V8
- U5 pad AA5: /RGMII PHY/RGMII_TXD1 -> /RGMII PHY/LA0_DQ3_P
- U5 pad AA6: /RGMII PHY/RGMII_TX_EN -> /RGMII PHY/LA0_DQ4_P
- U5 pad AA8: /RGMII PHY/ETH_RST_N -> /RGMII PHY/LA0_DQ0_N
- U5 pad AA9: /RGMII PHY/ETH_MDC -> /RGMII PHY/LA0_DQ0_P
- U5 pad AB10: /RGMII PHY/ETH_MDIO -> /RGMII PHY/LA0_DQ7_N
- U5 pad AB11: /RGMII PHY/LA0_DQ3_N -> /RGMII PHY/LA0_DQ2_N
- U5 pad AB12: /RGMII PHY/LA0_DQ5_N -> /RGMII PHY/RGMII_TX_CLK
- U5 pad AB13: /RGMII PHY/LA0_DQ5_P -> /RGMII PHY/RGMII_TXD3
- U5 pad AB5: /RGMII PHY/RGMII_TXD2 -> /RGMII PHY/LA0_DQ3_N
- U5 pad AB6: /RGMII PHY/ETH_LED1_N_1V8 -> /RGMII PHY/LA0_DQ4_N
- U5 pad AB7: /RGMII PHY/RGMII_TX_CLK -> /RGMII PHY/LA0_DQ5_N
- U5 pad AB8: /RGMII PHY/RGMII_TXD3 -> /RGMII PHY/LA0_DQ5_P
- U5 pad B1: /SERDES interfaces/GTX_TX2_N -> /SERDES interfaces/SFP_TX_N
- U5 pad B2: /SERDES interfaces/GTX_TX2_P -> /SERDES interfaces/SFP_TX_P
- U5 pad C10: /3.3V I/O/SFP_RX_LOS -> /3.3V I/O/PMOD_DQ1
- U5 pad C3: /SERDES interfaces/GTX_RX2_N -> /SERDES interfaces/SFP_RX_N
- U5 pad C4: /SERDES interfaces/GTX_RX2_P -> /SERDES interfaces/SFP_RX_P
- U5 pad D1: /SERDES interfaces/GTX_TX1_N -> /SERDES interfaces/GTX_TX2_P
- U5 pad D10: /3.3V I/O/SFP_RS1 -> /3.3V I/O/PMOD_DQ2
- U5 pad D11: /3.3V I/O/PMOD_DQ2 -> /3.3V I/O/SFP_RS1
- U5 pad D2: /SERDES interfaces/GTX_TX1_P -> /SERDES interfaces/GTX_TX2_N
- U5 pad D5: /SERDES interfaces/REFCLK_156_AC_N -> /SERDES interfaces/REFCLK_156_AC_P
- U5 pad D6: /SERDES interfaces/REFCLK_156_AC_P -> /SERDES interfaces/REFCLK_156_AC_N
- U5 pad E11: /3.3V I/O/PMOD_DQ1 -> /3.3V I/O/SFP_TX_DISABLE
- U5 pad E3: /SERDES interfaces/GTX_RX1_N -> /SERDES interfaces/GTX_RX2_N
- U5 pad E4: /SERDES interfaces/GTX_RX1_P -> /SERDES interfaces/GTX_RX2_P
- U5 pad F1: /SERDES interfaces/SFP_TX_N -> /SERDES interfaces/GTX_TX1_N
- U5 pad F11: /3.3V I/O/SFP_TX_DISABLE -> /3.3V I/O/SFP_RX_LOS
- U5 pad F13: /RAM_SDA -> /SERDES interfaces/SFP_I2C_SDA
- U5 pad F14: /3.3V I/O/SFP_RS0 -> /RAM_SDA
- U5 pad F2: /SERDES interfaces/SFP_TX_P -> /SERDES interfaces/GTX_TX1_P
- U5 pad F5: /SERDES interfaces/REFCLK_125_AC_N -> /SERDES interfaces/REFCLK_125_AC_P
- U5 pad F6: /SERDES interfaces/REFCLK_125_AC_P -> /SERDES interfaces/REFCLK_125_AC_N
- U5 pad G3: /SERDES interfaces/SFP_RX_N -> /SERDES interfaces/GTX_RX1_N
- U5 pad G4: /SERDES interfaces/SFP_RX_P -> /SERDES interfaces/GTX_RX1_P
- U5 pad H13: /SERDES interfaces/SFP_I2C_SDA -> /3.3V I/O/SFP_RS0
- U5 pad L21: /DDR/RAM_CK1_P -> /DDR/RAM_CK1_N
- U5 pad M20: /DDR/RAM_CK0_N -> /DDR/RAM_CK1_P
- U5 pad M21: /DDR/RAM_CK0_P -> /DDR/RAM_CK0_N
- U5 pad N20: /DDR/RAM_CKE0 -> /DDR/RAM_CK0_P
- U5 pad N5: /Expansion connector/LA1_DQ1_P -> /Expansion connector/LVDS15_P
- U5 pad P5: /Expansion connector/LA1_DQ1_N -> /Expansion connector/LVDS15_N
- U5 pad R18: /DDR/RAM_CK1_N -> /DDR/RAM_CKE0
- U5 pad R7: /RGMII PHY/ETH_RX_DV -> (no net)
- U5 pad T13: /RGMII PHY/LA0_DQ7_P -> /RGMII PHY/ETH_LED2_N_1V8
- U5 pad T5: /Expansion connector/LVDS15_P -> /Expansion connector/LA1_DQ1_P
- U5 pad T6: /RGMII PHY/RGMII_TXD0 -> (no net)
- U5 pad U11: /RGMII PHY/LA0_DQ0_N -> /RGMII PHY/ETH_RST_N
- U5 pad U12: /RGMII PHY/LA0_DQ0_P -> /RGMII PHY/ETH_MDC
- U5 pad U13: /RGMII PHY/LA0_DQ7_N -> /RGMII PHY/ETH_MDIO
- U5 pad U5: /Expansion connector/LVDS15_N -> /Expansion connector/LA1_DQ1_N
- U5 pad V12: /RGMII PHY/LA0_DQ6_N -> /RGMII PHY/ETH_RXD0
- U5 pad V13: /RGMII PHY/LA0_DQ6_P -> /RGMII PHY/ETH_RXD1
- U5 pad W12: /RGMII PHY/LA0_DQ2_P -> /RGMII PHY/RGMII_TXD1
- U5 pad W6: /RGMII PHY/ETH_RXD1 -> /RGMII PHY/LA0_DQ6_P
- U5 pad W9: (no net) -> /RGMII PHY/RGMII_TXD0
- U5 pad Y12: /RGMII PHY/LA0_DQ2_N -> /RGMII PHY/RGMII_TXD2
- U5 pad Y13: /RGMII PHY/LA0_DQ4_P -> /RGMII PHY/RGMII_TX_EN
- U5 pad Y6: /RGMII PHY/ETH_RXD0 -> /RGMII PHY/LA0_DQ6_N
- U5 pad Y9: (no net) -> /RGMII PHY/ETH_RX_DV
Routing:
- net /GND: track 0.00 -> 1246.3 mm, vias 0 -> 193
- net /1V35: track 0.00 -> 178.9 mm, vias 0 -> 36
- net /3V3: track 0.00 -> 131.6 mm, vias 0 -> 10
- net /1V8: track 0.00 -> 101.6 mm, vias 0 -> 24
- net /RAM_VREF: track 0.00 -> 79.5 mm, vias 0 -> 7
- net /SERDES interfaces/SFP_RX_P: track 0.00 -> 54.4 mm
- net /1V0: track 0.00 -> 54.3 mm, vias 0 -> 17
- net /SERDES interfaces/SFP_RX_N: track 0.00 -> 53.5 mm
- net /SERDES interfaces/SFP_TX_N: track 0.00 -> 49.9 mm, vias 0 -> 2
- net /SERDES interfaces/SFP_TX_P: track 0.00 -> 49.6 mm, vias 0 -> 2
- net /SERDES interfaces/GTX_RX3_P: track 0.00 -> 48.6 mm
- net /SERDES interfaces/GTX_RX3_N: track 0.00 -> 48.6 mm
- net /SERDES interfaces/GTX_TX3_N: track 0.00 -> 47.8 mm
- net /SERDES interfaces/GTX_TX3_P: track 0.00 -> 47.8 mm
- net /SERDES interfaces/GTX_RX2_P: track 0.00 -> 36.5 mm, vias 0 -> 1
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Other:
- net class Default: clearance 0.1 -> 0.07; trace_width 0.16 -> 0.1
- rule trace_clearance: 0.1 -> 0.07
- rule trace_min: 0.1 -> 0.07
- board text added: "12V DC"
- board text added: "3V3"
- board text added: "EXPANSION"
- board text added: "GND"
- board text added: "GPIO PMOD"
- board text added: "JTAG"
- board text added: "LA0"
- board text added: "LA1"
- board text added: "RX+"
- board text added: "RX-"
- board text added: "SATA DEVICE"
- board text added: "SATA HOST"
- board text added: "TX+"
- board text added: "TX-"

Commit message: Continued initial work on layout. BGA fanout and southwest area
Parts:
- C61: moved to B.Cu
- moved R61 225.8 mm to (57.8, 101.2)
- moved R62 222.6 mm to (56.8, 95.2)
- moved R52 218.9 mm to (39.6, 144.8)
- moved C113 217.8 mm to (58.8, 92.0)
- moved R47 217.7 mm to (55.7, 140.0)
- moved C115 216.8 mm to (64.5, 92.0)
- moved R51 215.7 mm to (44.6, 138.9)
- moved R50 212.3 mm to (46.0, 141.7)
- moved R4 210.7 mm to (56.8, 98.2)
- moved C99 210.3 mm to (48.6, 141.7)
- moved TP13 209.1 mm to (71.0, 137.0), turned to 180 degrees
- moved C103 206.2 mm to (43.3, 144.7)
- moved TP7 203.0 mm to (68.7, 67.0)
- moved TP3 200.9 mm to (55.2, 93.0)
- moved C102 198.1 mm to (47.5, 138.9)
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Connections:
- U5 pad K1: /Expansion connector/LVDS1_P -> /Expansion connector/LVDS0_P
- U5 pad K2: /Expansion connector/LVDS3_N -> /Expansion connector/LA1_DQ0_N
- U5 pad K3: /Expansion connector/LVDS3_P -> /Expansion connector/LA1_DQ0_P
- U5 pad L1: /Expansion connector/LVDS1_N -> /Expansion connector/LVDS0_N
- U5 pad L3: /Expansion connector/LVDS0_P -> /Expansion connector/LVDS1_P
- U5 pad L4: /Expansion connector/LVDS5_N -> /Expansion connector/LVDS14_N
- U5 pad L5: /Expansion connector/LVDS5_P -> /Expansion connector/LVDS14_P
- U5 pad M1: /Expansion connector/LVDS2_N -> /Expansion connector/LVDS2_P
- U5 pad M2: /Expansion connector/LVDS2_P -> /Expansion connector/LVDS2_N
- U5 pad M3: /Expansion connector/LVDS0_N -> /Expansion connector/LVDS1_N
- U5 pad M5: /Expansion connector/LVDS8_P -> /Expansion connector/LA1_DQ3_P
- U5 pad N2: /Expansion connector/LVDS4_N -> /Expansion connector/LVDS11_N
- U5 pad N3: /Expansion connector/LVDS4_P -> /Expansion connector/LVDS11_P
- U5 pad N4: /Expansion connector/LVDS8_N -> /Expansion connector/LA1_DQ3_N
- U5 pad P1: /Expansion connector/LVDS7_P -> /Expansion connector/LVDS3_P
- U5 pad P2: /Expansion connector/LVDS6_P -> /Expansion connector/LA1_DQ4_P
- U5 pad R1: /Expansion connector/LVDS7_N -> /Expansion connector/LVDS3_N
- U5 pad R2: /Expansion connector/LVDS6_N -> /Expansion connector/LA1_DQ4_N
- U5 pad R3: /Expansion connector/LVDS11_P -> /Expansion connector/LVDS4_P
- U5 pad T1: /Expansion connector/LVDS9_P -> /Expansion connector/LVDS5_P
- U5 pad T3: /Expansion connector/LVDS11_N -> /Expansion connector/LVDS4_N
- U5 pad U1: /Expansion connector/LVDS9_N -> /Expansion connector/LVDS5_N
- U5 pad U2: /Expansion connector/LVDS14_P -> /Expansion connector/LVDS6_P
- U5 pad V2: /Expansion connector/LVDS14_N -> /Expansion connector/LVDS6_N
- U5 pad V3: /Expansion connector/LA1_DQ0_P -> /Expansion connector/LVDS7_P
- U5 pad W1: /Expansion connector/LA1_DQ3_P -> /Expansion connector/LVDS8_P
- U5 pad W2: /Expansion connector/LA1_DQ0_N -> /Expansion connector/LVDS7_N
- U5 pad Y1: /Expansion connector/LA1_DQ3_N -> /Expansion connector/LVDS8_N
- U5 pad Y2: /Expansion connector/LA1_DQ4_N -> /Expansion connector/LVDS9_P
- U5 pad Y3: /Expansion connector/LA1_DQ4_P -> /Expansion connector/LVDS9_N
Routing:
- net /GND: track 1246.3 -> 1360.9 mm, vias 193 -> 227
- net /FPGA power/GTX_1V8: track 0.71 -> 73.0 mm, vias 1 -> 12
- net /1V2: track 0.00 -> 50.0 mm, vias 0 -> 5
- net /GTX_1V2: track 14.1 -> 63.0 mm, vias 5 -> 17
- net /1V0: track 54.3 -> 97.8 mm, vias 17 -> 21
- net /FPGA power/GTX_1V0: track 10.2 -> 46.6 mm, vias 4 -> 9
- net /1V8: track 101.6 -> 134.8 mm, vias 24 -> 29
- net /Expansion connector/LVDS9_N: track 3.93 -> 26.8 mm
- net /Expansion connector/LVDS7_P: track 3.92 -> 26.3 mm
- net /Expansion connector/LVDS2_N: track 2.72 -> 25.0 mm
- net /Expansion connector/LVDS1_P: track 3.33 -> 25.5 mm
- net /Expansion connector/LVDS1_N: track 3.41 -> 25.5 mm
- net /Expansion connector/LVDS9_P: track 4.01 -> 25.8 mm
- net /Expansion connector/LVDS6_P: track 3.58 -> 25.1 mm, vias 1 -> 0
- net /Expansion connector/LVDS6_N: track 3.58 -> 25.1 mm, vias 1 -> 0
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Other:
- board text added: "1V0"
- board text added: "1V2"
- board text added: "G1V2"
- board text added: "G1V8"

Commit message: Continued routing for tonight. Bunch of low speed stuff in south area of board.
Parts:
- C102, C103, C55, C63, C64, C65, C66, C67, R28, R29, R33, R34, R45, R46, R47, R48, R49: moved to B.Cu
- moved TP17 85.0 mm to (71.0, 137.0), turned to 180 degrees
- moved C55 57.7 mm to (108.7, 113.0), turned to 270 degrees
- moved TP1 49.0 mm to (81.0, 108.8)
- moved TP2 44.5 mm to (86.4, 109.8)
- moved R52 39.3 mm to (57.5, 109.8)
- moved TP13 37.5 mm to (83.4, 101.7)
- moved L5 37.2 mm to (62.0, 112.6), turned to 90 degrees
- moved C98 36.8 mm to (63.9, 111.7)
- moved R50 35.7 mm to (63.9, 110.8)
- moved C101 33.7 mm to (58.0, 112.5), turned to 90 degrees
- moved R51 33.2 mm to (60.6, 109.8), turned to 180 degrees
- moved C100 33.2 mm to (60.1, 112.5), turned to 90 degrees
- moved C99 30.5 mm to (54.2, 111.7), turned to 180 degrees
- moved L6 28.9 mm to (56.1, 112.5), turned to 90 degrees
- moved C103 28.4 mm to (57.9, 120.3), turned to 180 degrees
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Connections:
- C34 pad 1: /SERDES interfaces/GTX_RX3_P -> /SERDES interfaces/GTX_TX3_P
- C35 pad 1: /SERDES interfaces/GTX_RX3_N -> /SERDES interfaces/GTX_TX3_N
- C36 pad 1: /SERDES interfaces/GTX_TX3_P -> /SERDES interfaces/GTX_RX3_P
- C36 pad 2: /SERDES interfaces/GTX_TX3_AC_P -> /SERDES interfaces/GTX_RX3_AC_P
- C37 pad 1: /SERDES interfaces/GTX_TX3_N -> /SERDES interfaces/GTX_RX3_N
- C37 pad 2: /SERDES interfaces/GTX_TX3_AC_N -> /SERDES interfaces/GTX_RX3_AC_N
- J2 pad 1: /SERDES interfaces/GTX_TX3_P -> /SERDES interfaces/GTX_RX3_AC_P
- J5 pad 1: /SERDES interfaces/GTX_TX3_N -> /SERDES interfaces/GTX_RX3_AC_N
- J6 pad 1: /SERDES interfaces/GTX_RX3_P -> /SERDES interfaces/GTX_TX3_AC_P
- J7 pad 1: /SERDES interfaces/GTX_RX3_N -> /SERDES interfaces/GTX_TX3_AC_N
- U5 pad A10: /3.3V I/O/LA1_UART_TX -> /3.3V I/O/ETH_LED1_P
- U5 pad A11: /3.3V I/O/LA1_PRESENCE_DETECT -> /3.3V I/O/PMOD_DQ1
- U5 pad A8: /3.3V I/O/LA0_PRESENCE_DETECT -> /3.3V I/O/LED0
- U5 pad A9: /3.3V I/O/LA1_12V0_EN -> /3.3V I/O/LED3
- U5 pad AB12: /RGMII PHY/RGMII_TX_CLK -> /RGMII PHY/LA0_DQ1_N
- U5 pad AB13: /RGMII PHY/RGMII_TXD3 -> /RGMII PHY/LA0_DQ1_P
- U5 pad B10: /3.3V I/O/LA0_12V0_EN -> /3.3V I/O/PMOD_DQ7
- U5 pad B11: /3.3V I/O/LA1_12V0_FAULT -> /3.3V I/O/LED1
- U5 pad B8: /3.3V I/O/LA0_UART_RX -> /3.3V I/O/LA1_12V0_FAULT
- U5 pad C10: /3.3V I/O/PMOD_DQ1 -> /3.3V I/O/LA1_PRESENCE_DETECT
- U5 pad C8: /3.3V I/O/LA0_UART_TX -> /3.3V I/O/LA1_UART_TX
- U5 pad C9: /3.3V I/O/LA0_12V0_FAULT -> /3.3V I/O/LA0_12V0_EN
- U5 pad D9: /3.3V I/O/LED3 -> /3.3V I/O/LA1_12V0_EN
- U5 pad E9: /3.3V I/O/ETH_LED1_P -> /3.3V I/O/LA0_12V0_FAULT
- U5 pad F8: /3.3V I/O/LED1 -> /3.3V I/O/LA0_UART_RX
- U5 pad F9: /3.3V I/O/PMOD_DQ7 -> /3.3V I/O/LA0_UART_TX
- U5 pad G8: /3.3V I/O/LED0 -> /3.3V I/O/LA0_PRESENCE_DETECT
- U5 pad K2: /Expansion connector/LA1_DQ0_N -> /Expansion connector/LVDS11_N
- U5 pad K3: /Expansion connector/LA1_DQ0_P -> /Expansion connector/LVDS11_P
- U5 pad L4: /Expansion connector/LVDS14_N -> /Expansion connector/LVDS10_N
- U5 pad L5: /Expansion connector/LVDS14_P -> /Expansion connector/LVDS10_P
- U5 pad M5: /Expansion connector/LA1_DQ3_P -> /Expansion connector/LVDS12_P
- U5 pad N2: /Expansion connector/LVDS11_N -> /Expansion connector/LVDS13_N
- U5 pad N3: /Expansion connector/LVDS11_P -> /Expansion connector/LVDS13_P
- U5 pad N4: /Expansion connector/LA1_DQ3_N -> /Expansion connector/LVDS12_N
- U5 pad N5: /Expansion connector/LVDS15_P -> /Expansion connector/LVDS14_P
- U5 pad P2: /Expansion connector/LA1_DQ4_P -> /Expansion connector/LVDS15_P
- U5 pad P4: /Expansion connector/LVDS10_P -> /Expansion connector/LA1_DQ4_P
- U5 pad P5: /Expansion connector/LVDS15_N -> /Expansion connector/LVDS14_N
- U5 pad R2: /Expansion connector/LA1_DQ4_N -> /Expansion connector/LVDS15_N
- U5 pad R4: /Expansion connector/LVDS10_N -> /Expansion connector/LA1_DQ4_N
- U5 pad T4: /Expansion connector/LVDS12_P -> /Expansion connector/LA1_DQ3_P
- U5 pad T8: /RGMII PHY/LA0_DQ1_N -> /RGMII PHY/RGMII_TX_CLK
- U5 pad T9: /RGMII PHY/LA0_DQ1_P -> /RGMII PHY/RGMII_TXD3
- U5 pad U3: /Expansion connector/LVDS12_N -> /Expansion connector/LA1_DQ3_N
- U5 pad V4: /Expansion connector/LVDS13_P -> /Expansion connector/LA1_DQ0_P
- U5 pad W4: /Expansion connector/LVDS13_N -> /Expansion connector/LA1_DQ0_N
Routing:
- net /GND: track 1360.9 -> 1644.0 mm, vias 227 -> 260
- net /FPGA support/JTAG_TDI: track 0.71 -> 103.9 mm, vias 1 -> 4
- net /FPGA support/JTAG_TCK: track 0.71 -> 103.9 mm, vias 1 -> 2
- net /FPGA support/JTAG_TMS: track 0.71 -> 98.2 mm, vias 1 -> 2
- net /3.3V I/O/LA1_PRESENCE_DETECT: track 1.50 -> 46.6 mm, vias 0 -> 2
- net /3V3: track 131.6 -> 176.0 mm, vias 10 -> 13
- net /3.3V I/O/LA1_12V0_FAULT: track 2.71 -> 46.0 mm, vias 0 -> 2
- net /3.3V I/O/LA1_UART_TX: track 1.50 -> 42.6 mm, vias 0 -> 2
- net /FPGA power/GTX_1V0: track 46.6 -> 86.8 mm, vias 9 -> 11
- net /3.3V I/O/LA1_12V0_EN: track 1.50 -> 38.2 mm, vias 0 -> 2
- net /3.3V I/O/LA0_12V0_EN: track 2.71 -> 39.2 mm, vias 0 -> 2
- net /3.3V I/O/LA0_12V0_FAULT: track 0.71 -> 37.0 mm, vias 1 -> 2
- net /Expansion connector/LVDS11_N: track 4.71 -> 39.2 mm, vias 1 -> 2
- net /Expansion connector/LVDS11_P: track 5.01 -> 39.2 mm, vias 1 -> 2
- net /Expansion connector/LVDS13_N: track 5.38 -> 39.2 mm, vias 1 -> 2
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Other:
- board text added: "G1V0"
- board text removed: "1V0"
